File: pcb/mcu.kicad_sch (KiCad schematic)
At the start: 1 part, among them U1 ESP32-S3-MINI-1

Commit message: Added Pins to MCU sheet Signed-off-by: Damir Gazizullin <dgazizul@uwaterloo.ca>
Parts:
- added C83, C85, C86: 270nF ±10% X7R 0402, Capacitor_SMD:C_0402_1005Metric, symbol Device:C_Small
- added C84: 22uF ±10% X5R 0805, Capacitor_SMD:C_0805_2012Metric, symbol Device:C_Small
- added R79, R80, R81, R82: 4.7kΩ ±1%, Resistor_SMD:R_0402_1005Metric, symbol Device:R_Small_US
- added SW2, SW3: TS-1088-AR02016, TS-1088-AR02016:SW-SMD_L3.9-W3.0-P4.45, symbol TS-1088-AR02016:TS-1088-AR02016
Connections:
- net GND: now reaches U1.1 (GND), U1.2 (GND), U1.42 (GND), U1.43 (GND), U1.46 (GND), U1.47 (GND), U1.48 (GND), U1.49 (GND), U1.50 (GND), U1.51 (GND), U1.52 (GND), U1.53 (GND), U1.54 (GND), U1.55 (GND), U1.56 (GND), U1.57 (GND), U1.58 (GND), U1.59 (GND), U1.60 (GND), U1.61 (GND), U1.62 (GND), U1.63 (GND), U1.64 (GND), U1.65 (GND)
- net GND: now also C83.2, C84.2, C85.2, C86.2, SW2.2, SW3.2
- net +3.3V: now reaches U1.3 (3V3)
- net +3.3V: now also C83.1, C84.1, R80.1, R82.1
- net BOOT_MODE: now reaches U1.4 (IO0)
- net BOOT_MODE: now also C86.1, R81.1
- net ESP32_EN: now reaches U1.45 (EN)
- net ESP32_EN: now also C85.1, R79.1
- new net: R81.2, R82.2, SW3.1
- new net: R79.2, R80.2, SW2.1
Other:
- moved on the sheet: U1
